File: resistance_board_RE/resistance_board_RE.kicad_sch (KiCad schematic)
At the start: 6 parts, among them J1 Red Wire, Q1 FZT658

Commit message: asdf
Parts:
- added C1, C2: 100nF Film, symbol Device:C
- added C3: C, symbol Device:C
- added D1: BAV99, Package_TO_SOT_SMD:SOT-23, symbol Diode:BAV99
- added J2: Blrown Wire, symbol Connector_Generic:Conn_01x01
- added J3: Yellow Wire, symbol Connector_Generic:Conn_01x01
- added J4: Black Wire, symbol Connector_Generic:Conn_01x01
- added L3, L4: 220k, symbol Device:L
- added Q2: SOT_23 Device "GM X", symbol Device:Q_NPN_BCE
- added Q3: 04N80C3, symbol Device:Q_NMOS_GDS
- added Q4: FZT758, symbol Device:Q_PNP_BCE
- added Q5: TIP32CG Heatsunk, symbol Device:Q_PNP_BCE
- added Q6: Q_PMOS_GDS, symbol Device:Q_PMOS_GDS
- added R10, R11, R12, R13, R9: 68k, symbol Device:R
- added R14: 1k, symbol Device:R
- added R3, R4: 10M, symbol Device:R
- added R5, R6, R7, R8: 100k, symbol Device:R
- added RL102: TX2-L-12V, symbol Relay:G6KU-2
- added TP102: TestPoint, symbol Connector:TestPoint
- added U1, U3: PVI5080N, VOM1271T:SOIC254P695X242-4N, symbol vom1271:PVI5080N
- added U2: LTC1052CSW-PBF, SO-16_SW_LIT, symbol ltc1052:LTC1052CSW-PBF
- added U4: LTC1150, symbol Amplifier_Operational:LTC1152
Connections:
- net at Q1.2 (C): now also Q3.2 (D)
- new net: L3.2, L4.1, R3.2, R4.1
- new net: L4.2, Q4.1 (B), Q4.3 (E), R4.2
- new net: L3.1, R3.1, R5.2, RL102.5, TP102.1
- new net: Q3.1 (G), U1.5
- new net: C3.1, Q6.1 (G), U3.8
- new net: C3.2, D1.1 (K), D1.2 (A), R14.1, U3.5
- new net: D1.3 (K), R13.1, R14.2
- new net: R12.1, R13.2
- new net: R11.1, R12.2
- new net: R6.1, R7.2
- new net: R5.1, R6.2
- new net: J2.1 (Pin_1), Q2.2 (C)
- new net: J3.1 (Pin_1), U2.3 (NC(GUARD)), U2.5 (+IN), U2.6 (NC(GUARD))
- new net: Q5.2 (C), R8.1
- new net: R7.1, R8.2
- new net: RL102.3, RL102.6
- new net: J4.1 (Pin_1), RL102.4
- new net: C1.1, C2.1, U2.10 (CRETURN)
- new net: C1.2, U2.1 (CEXTB)
- new net: Q4.2 (C), Q6.2 (D), R9.2
- new net: C2.2, U2.2 (CEXTA)
- new net: R10.1, R11.2
- new net: R10.2, R9.1

Commit message: asdf
Parts:
- added C4, C5, C6, C7, C8, C9: C, symbol Device:C
- added NT1, NT10, NT11, NT12, NT2, NT3, NT4, NT5, NT6, NT7, NT8, NT9: NetTie_2, symbol Device:NetTie_2
- added Q10: MMBF5485 "6M", symbol Device:Q_NJFET_DSG
- added Q7: BC856 "3DW", symbol Device:Q_PNP_BEC
- added Q8: TIP31AG Heatsunk, symbol Device:Q_NPN_BCE
- added Q9: BC846 "1DW", symbol Device:Q_NPN_BEC
- added R15, R21, R23: 100k, symbol Device:R
- added R16, R22: 1k, symbol Device:R
- added R17, R20: 40R, symbol Device:R
- added R18: 200R, symbol Device:R
- added R19: 2k, symbol Device:R
- added U5: DG211, Package_SO:SOIC-16_3.9x9.9mm_P1.27mm, symbol Analog_Switch:DG411xY
- added U7: LTC1150, symbol Amplifier_Operational:LTC1152
Connections:
- net at U4.2 (-): now also C6.2, R16.2
- net at U4.3 (+): now also U5.11
- net at U4.4 (V-): now also C4.1, Q7.3 (C)
- net at U4.6: now also C6.1, Q7.1 (B)
- net at U4.7 (V+): now also C5.1
- net at Q5.1 (B): now also R15.1
- net at Q5.3 (E): now also NT4.2, Q7.2 (E), R15.2
- new net: NT10.1, NT9.1, R18.1
- new net: NT11.1, NT12.1, R18.2
- new net: C9.1, U7.4 (V-)
- new net: Q8.1 (B), Q9.2 (E), R23.1
- new net: Q8.3 (E), R21.2, R23.2
- new net: C7.1, Q10.3 (G), U7.6
- new net: C7.2, R22.2, U7.2 (-)
- new net: NT5.1, NT8.1, R19.1
- new net: NT6.1, NT7.1, R19.2
- new net: NT2.1, NT3.1, R17.2, R20.2
- new net: NT2.2, R22.1
- new net: NT1.1, NT4.1, R17.1, R20.1
- new net: Q10.1 (D), Q9.3 (C)
- new net: Q10.2 (S), Q9.1 (B), R21.1
- new net: NT7.2, U7.3 (+)
- new net: C8.1, U7.7 (V+)
- new net: NT1.2, R16.1
- new net GND: C4.2, C5.2, C8.2, C9.2
Other:
- note added: "RN1 Fluke 4345146R"
- moved on the sheet: Q5, U4

Commit message: asdf
Parts:
- removed Q2: SOT_23 Device "GM X", symbol Device:Q_NPN_BCE
- added J5: Green Wire, symbol Connector_Generic:Conn_01x01
- added Q11: MMBF5485 "6M", symbol Device:Q_NJFET_DSG
- added R24: 100k, symbol Device:R
- added R25: 1M, symbol Device:R
- added RL101: TX2-L-12V, symbol Relay:G6KU-2
Connections:
- net at L3.1, R3.1, R5.2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: now also RL101.5
- net at J2.1 (Pin_1): now also Q11.2 (S)
- new net: R24.1, R25.2, RL101.2, RL101.3, RL101.6
- new net: Q11.1 (D), R24.2
Other:
- moved on the sheet: J2

Commit message: asdf
Parts:
- added C1, C2: C, symbol Device:C
- added D2, D5, D7: BAS21 "JS t", Package_TO_SOT_SMD:SOT-23, symbol Diode:BAS21
- added D3: BZX84C6V2 "WB1", Package_TO_SOT_SMD:SOT-23, symbol Diode:BZX84Cxx
- added D4: BZX84C8V2 "Z7W", Package_TO_SOT_SMD:SOT-23, symbol Diode:BZX84Cxx
- added D6: D_Schottky, symbol Device:D_Schottky
- added M104: MC33071, symbol Amplifier_Operational:OP07
- added Q12: BC856 "3DW", symbol Device:Q_PNP_BEC
- added Q13: FZT493, symbol Device:Q_NPN_BCE
- added Q14, Q2: TIP32CG Heatsunk, symbol Device:Q_PNP_BCE
- added R26, R27: 100k, symbol Device:R
- added R28: 1k, symbol Device:R
- added R29: 10k, symbol Device:R
- added R30: 1.5k, symbol Device:R
- added R31: 10.2k, symbol Device:R
- added TP1: TestPoint, symbol Connector:TestPoint
- added U2: LM337_TO220, Package_TO_SOT_THT:TO-220-3_Vertical, symbol Regulator_Linear:LM337_TO220
- renumbered C2 to C109, C1 to C110, U2 to M103
Connections:
- net GND: now also C1.1, C2.2, Q2.2 (C), R29.1, TP1.1
- new net: R26.1, R27.2
- new net: D2.1 (A), M104.6, R26.2
- new net: C1.2, D4.1 (A), M104.4 (V-)
- new net: C2.1, M104.7 (V+), Q12.1 (B), R29.2
- new net: D2.3 (K), Q13.2 (C), Q2.1 (B)
- new net: D5.3 (K), Q2.3 (E)
- new net: D4.3 (K), U2.3 (VO)
- new net: D5.1 (A), D6.1 (K)
- new net: D6.2 (A), D7.1 (A), Q14.1 (B)
- new net: Q12.2 (E), R30.1, R31.1
- new net: R27.1, R28.2
- new net: D3.3 (K), R30.2, R31.2
Other:
- moved on the sheet: C109, C110, J3, M103

Commit message: asdf
Parts:
- added C10: 10µF Tantal, symbol Device:C_Polarized
- added C11, C12, C13: 47nF Foil, symbol Device:C
- added D8: BZX84-C5V6 "Z3W", Package_TO_SOT_SMD:SOT-23, symbol Diode:BZX84Cxx
- added Q15: FZT658, symbol Device:Q_NPN_BCE
- added R32: 1k, symbol Device:R
- added R33: 2.2k, symbol Device:R
- added R34: 10M, symbol Device:R
Connections:
- net GND: now also R33.1
- net at R28.1: now also C10.2, C11.1, C12.1, R34.2
- net at Q13.1 (B): now also D8.3 (K), Q15.1 (B), R33.2
- net at Q13.3 (E): now also R32.2
- new net: D8.1 (A), R32.1
Other:
- moved on the sheet: D5, D6, D7, Q13, Q14, Q2

Commit message: asdf
Parts:
- removed D7: BAS21 "JS t", Package_TO_SOT_SMD:SOT-23, symbol Diode:BAS21
- added C14, C15, C16: C, symbol Device:C
- added D10, D11, D7: BAV99 "A7W", Package_TO_SOT_SMD:SOT-23, symbol Diode:BAV99
- added D9: BAV99 "JYW", Package_TO_SOT_SMD:SOT-23, symbol Diode:BAV99
- added Q104: SST404, Package_SO:SOIC-8_3.9x4.9mm_P1.27mm, symbol Transistor_FET:JFE2140D
- added Q16: BC856 "3DW", symbol Device:Q_PNP_BEC
- added Q17, Q18, Q19, Q20, Q22: BC846 "1DW", symbol Device:Q_NPN_BEC
- added Q21: FZT758, symbol Device:Q_PNP_BCE
- added R35: 100, symbol Device:R
- added R36, R37, R42, R46, R47, R48, R49: 47k, symbol Device:R
- added R38: 1k, symbol Device:R
- added R39, R53, R54: 4.7k, symbol Device:R
- added R40, R41: 2.2R, symbol Device:R
- added R43: 100R, symbol Device:R
- added R44, R51: 10k, symbol Device:R
- added R45: 22k, symbol Device:R
- added R50: 680k, symbol Device:R
- added R52: 2.2k, symbol Device:R
- added R55: 10M, symbol Device:R
- added TP2: TestPoint, symbol Connector:TestPoint
- added U6, U9: TL071, symbol Amplifier_Operational:TL071
- added U8: LTC1150, Package_SO:SOIC-8_3.9x4.9mm_P1.27mm, symbol Amplifier_Operational:LTC1152
Connections:
- net GND: now also U3.3, R45.2, R52.1
- net at M104.3 (+): now also D9.2 (A)
- net at C10.2, C11.1, C12.1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: now also D9.3 (K)
- net at D1.3 (K), R13.1, R14.2: now also Q21.1 (B), Q21.3 (E)
- net at D6.2 (A): now also Q14.2 (C); no longer Q14.1 (B)
- net at C10.1: now also R35.2, R36.2, R37.2
- net at Q14.3 (E): now also Q16.1 (B), R41.2
- new net: Q16.2 (E), R40.2, R43.1
- new net: C14.2, Q16.3 (C), R38.2, R39.1
- new net: D7.1 (K), Q20.2 (E), R49.1
- new net: Q17.1 (B), Q18.3 (C), R42.1, R49.2
- new net: R40.1, R41.1
- new net: Q19.3 (C), R43.2
- new net: R44.1, U8.6
- new net: D7.3 (K), Q18.1 (B), R46.1
- new net: Q20.1 (B), R47.2
- new net: Q20.3 (C), R48.1
- new net: R44.2, R45.1, U6.3 (+)
- new net: R51.1, R52.2
- new net: C15.2, C16.2, D11.1 (K), Q22.3 (C), R54.1, R55.1
- new net: C15.1, C16.1, R53.1, R54.2, R55.2
- new net: Q14.1 (B), R38.1
- new net: R50.1, R51.2, R53.2, U9.3 (+)
- new net: Q19.1 (B), U6.6
- new net: Q19.2 (E), R42.2, TP2.1, U6.2 (-)
- new net: Q17.2 (E), R48.2
- new net: C14.1, Q17.3 (C), R39.2
- new net: D10.3 (K), R46.2, R47.1, U9.6
- new net: Q21.2 (C), Q22.2 (E)
- new net: D10.2 (A), R50.2
- no-connect marks 0 -> 3
Other:
- note added: "1V"
- note added: "7.5V"
- note added: "8.19V"
- note added: "Hot"
- moved on the sheet: C1, C10, C109, C11, C110, C12, C13, C2, C3, C4, C5, C6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

Commit message: asdf
Parts:
- added C17, C21: C, symbol Device:C
- added C18: 3.3nF Foil, symbol Device:C
- added C19, C20: 10nF Foil, symbol Device:C
- added C22, C23: 10µF Tantal, symbol Device:C_Polarized
- added D12, D13, D14: BAV99 "A7W", Package_TO_SOT_SMD:SOT-23, symbol Diode:BAV99
- added J6: Orange Wire, symbol Connector_Generic:Conn_01x01
- added M203: LTC1052CSW-PBF, SO-16_SW_LIT, symbol ltc1052:LTC1052CSW-PBF
- added NT13: NetTie_2, symbol Device:NetTie_2
- added Q23: BC856 "3DW", symbol Device:Q_PNP_BEC
- added Q24: BC846 "1DW", symbol Device:Q_NPN_BEC
- added R104: 27k, symbol Device:R
- added R56, R57: 47k, symbol Device:R
- added R58, R59, R60, R61: 2.7k, symbol Device:R
- added R62: 1k, symbol Device:R
- added R63, R64, R65, R66, R67: 68k, symbol Device:R
- added R68, R69: 10k, symbol Device:R
- added RL104, RL2: TX2-L-12V, symbol Relay:G6KU-2
- added TP3: TestPoint, symbol Connector:TestPoint
- added U10: TL071, symbol Amplifier_Operational:TL071
- D1: value BAV99 -> BAV99 "A7W"
Connections:
- net GND: now also D7.1 (K), Q20.2 (E), R49.1, U1.3, C22.1, C23.2, D12.1 (K), D14.2 (A), RL104.4, RL2.5, RL2.6, RL2.7, RL2.8
- net at C10.2, C11.1, C12.1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: now also J5.1 (Pin_1)
- net at U1.2: now also R58.2, R59.2
- net at Q3.1 (G), U1.5: now also C17.2
- net at U1.8: now also C17.1, D13.3 (K), R62.2
- net at Q18.2 (E): now also Q17.2 (E), R48.2
- net at Q20.1 (B), R47.2: now also D12.2 (A)
- net at U3.2: now also R60.2, R61.2
- net at C16.2, D11.1 (K), R55.1: now also U9.2 (-), U10.2 (-); no longer C15.2, Q22.3 (C), R54.1
- net at C15.1, C16.1, R53.1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: now also Q23.2 (E), R56.1
- net at Q1.2 (C), Q3.2 (D): now also R67.1
- net at Q3.3 (S): now also RL104.5, TP3.1
- net at D11.3 (K): now also U10.6
- new net: Q24.1 (B), Q24.2 (E), R69.1
- new net: M203.3 (NC(GUARD)), M203.4 (-IN), R68.1, R69.2
- new net: NT13.1, RL104.6
- new net: C21.1, NT13.2, Q24.3 (C)
- new net: R56.2, R57.2
- new net: R65.1, R67.2
- new net: C18.1, R104.1, RL104.2, RL2.4
- new net: RL104.3, RL104.7
- new net: C22.2, D14.1 (K)
- new net: J6.1 (Pin_1), R104.2
- new net: R65.2, R66.1
- new net: R64.1, R66.2
- new net: C18.2, C19.2, C20.2
- new net: C21.2, D14.3 (K), R68.2
- new net: R63.1, R64.2
- new net: C15.2, Q22.3 (C), R54.1, U10.3 (+)
- new net: D13.1 (K), D13.2 (A), R62.1, R63.2
- new net +15V: R58.1, R59.1, R60.1, R61.1
- no-connect marks 3 -> 4
Other:
- note added: "Composite Amplifier "Low Follower""
- note added: "Constant current sinks maybe?"
- note added: "PSU region probably"
- note added: "Vref region probably"
- moved on the sheet: C1, C10, C109, C11, C110, C12, C13, C14, C15, C16, C2, C3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

Commit message: asdf
Parts:
- added R70, R72, R73, R74: 100k, symbol Device:R
- added R71: 4.7k, symbol Device:R
- added RL1: TX2-L-12V, symbol Relay:G6KU-2
- added U11: TL071, symbol Amplifier_Operational:TL071
Connections:
- net -15V: now reaches D8.1 (A), R32.1
- net -15V: now also R71.2
- net at Q15.2 (C): now also RL1.2
- net at Q15.3 (E): now also R71.1
- new net: RL1.3, RL1.7
- new net: R70.1, RL1.6
- new net: R70.2, R72.1
- new net: R72.2, R73.1, R74.1
- new net: R73.2, R74.2, U11.3 (+)
- no-connect marks 4 -> 5
Other:
- moved on the sheet: D8, Q13, Q15, R32, R33
