File: resistance_board_RE/resistance_board_RE.kicad_sch (KiCad schematic)
At the start: 200 parts, among them J1 Red Wire, J2 Blrown Wire, J3 Yellow Wire, J4 Black Wire, J5 Green Wire, J6 Orange Wire, M103 LTC1052CSW-PBF, M104 MC33071, M203 LTC1052CSW-PBF, Q1 FZT658, Q10 MMBF5485 "6M", Q104 SST404, Q11 MMBF5485 "6M", Q12 BC856 "3DW", Q13 FZT493, Q14 TIP32CG Heatsunk, Q15 FZT658, Q16 BC856 "3DW", Q17 BC846 "1DW", Q18 BC846 "1DW", Q19 BC846 "1DW", Q2 TIP32CG Heatsunk, Q20 BC846 "1DW", Q21 FZT758, Q22 BC846 "1DW", Q23 BC856 "3DW", Q24 BC846 "1DW", Q25 FZT493, Q26 BC846 "1DW", Q27 BC846 "1DW", Q28 BC846 "1DW", Q3 04N80C3, Q4 FZT758, Q5 TIP32CG Heatsunk, Q6 Q_PMOS_GDS, Q7 BC856 "3DW", Q8 TIP31AG Heatsunk, Q9 BC846 "1DW", U1 PVI5080N, U10 TL071, U11 TL071, U12 TL071, U2 LM337_TO220, U3 PVI5080N, U4 LTC1150, U5 DG211, U6 TL071, U7 LTC1150, U8 LTC1150, U9 TL071

Commit message: asdf
Parts:
- added C24: C, symbol Device:C
- added D16: BAV99 "JYW", Package_TO_SOT_SMD:SOT-23, symbol Diode:BAV99
- added Q29: FZT758, symbol Device:Q_PNP_BCE
- added Q30, Q31: Q_NJFET_DSG, symbol Device:Q_NJFET_DSG
- added R83, R84, R85, R86: 1M, symbol Device:R
- added R87, R89: 100k, symbol Device:R
- added R88: 10k, symbol Device:R
- added RL4, RL5: TX2-L-12V, symbol Relay:G6KU-2
Connections:
- net +15V: now also D16.2 (A)
- net at L3.1, R3.1, R5.2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: now also RL4.2
- net at C10.2, C11.1, C12.1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: now also R87.1
- net at C18.1, R104.1, RL104.2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: now also Q30.3 (G), Q31.1 (D), Q31.2 (S)
- net at Q27.2 (E), U11.2 (-): now also Q31.3 (G), R88.2
- new net: R84.2, R85.1
- new net: R85.2, R86.1
- new net: Q29.1 (B), Q29.3 (E), RL4.6
- new net: Q29.2 (C), Q30.1 (D), Q30.2 (S), R87.2
- new net: D16.3 (K), R86.2
- new net: R83.1, RL4.3, RL5.2
- new net: R88.1, R89.2
- new net: C24.2, RL4.5
- new net: R83.2, R84.1
Other:
- note added: "Compliance Voltage Clamping maybe?"
- note added: "~0V"
- note removed: "Constant current sinks maybe?"
- moved on the sheet: RL102, TP102

Commit message: asdf
Parts:
- added D17: BAV99 "A7W", Package_TO_SOT_SMD:SOT-23, symbol Diode:BAV99
- added D18: BZX84C6V2 "WB1", Package_TO_SOT_SMD:SOT-23, symbol Diode:BZX84Cxx
- added Q32: BC856 "3DW", symbol Device:Q_PNP_BEC
- added R90, R93: 1M, symbol Device:R
- added R91: 1k, symbol Device:R
- added R92: 10M, symbol Device:R
- added R94: 100k, symbol Device:R
- added R95: 180R, symbol Device:R
- added R96: 2.2k, symbol Device:R
Connections:
- net +15V: now also D18.3 (K), R94.1, R95.2
- net at D5.1 (A), D6.1 (K): now also D17.2 (A)
- net at RL5.3: now also RL5.6
- net at RL5.4: now also RL5.5, R90.1
- net at RL4.1: now also RL102.8
- new net: D18.1 (A), R96.1
- new net: Q32.1 (B), R94.2
- new net: R90.2, R91.1
- new net: R91.2, R92.1, R93.1
- new net: Q32.2 (E), R95.1, R96.2
- new net: D17.1 (K), Q32.3 (C)
Other:
- moved on the sheet: D15

Commit message: asdf
Parts:
- removed R89: 100k, symbol Device:R
- added R100, R101, R102: 100k, symbol Device:R
- added R97: 6.8k, symbol Device:R
- added R98: 68k, symbol Device:R
- added R99: 10k, symbol Device:R
- added U13: DG408DY+T, 21-0041T_S16+5_MXM, symbol dg408:DG408DY+T
- added U14: DG211, Package_SO:SOIC-16_3.9x9.9mm_P1.27mm, symbol Analog_Switch:DG411xY
- added unit 3 of U4
Connections:
- net -15V: now also R88.1, R101.2, R102.2
- net at Q15.2 (C), RL1.2: now also R97.1, R98.1
- net at R73.2, R74.2, U11.3 (+): now also R100.2
- new net: R98.2, R99.1
- new net: R100.1, R101.1, R102.1
- new net: U13.10 (S7), U13.11 (S6), U13.12 (S5), U13.4 (S1), U13.9 (S8)
- new net: R99.2, U14.3
- new net: U14.2, U4.10
Other:
- moved on the sheet: R34, R70, R72, R73, R74, R88

Commit message: asdf
Parts:
- removed Q30, Q31: Q_NJFET_DSG, symbol Device:Q_NJFET_DSG
- added D19: BAV99 "JYW", Package_TO_SOT_SMD:SOT-23, symbol Diode:BAV99
- added Q30, Q33: MMBF4117, symbol Device:Q_NJFET_SDG
- added Q31: FZT493, symbol Device:Q_NPN_BCE
- added Q34: BC846 "1DW", symbol Device:Q_NPN_BEC
- added R103: 22k, symbol Device:R
- added R105: 47k, symbol Device:R
- added R106: 2.2k, symbol Device:R
- added R107: 10k, symbol Device:R
- added R108, R89: 4.7k, symbol Device:R
- added U15: TL071, symbol Amplifier_Operational:TL071
Connections:
- net -15V: now also D19.2 (A), R108.2
- net GND: now also Q31.2 (C), U15.3 (+)
- net at U8.2 (-): now also R44.1, R105.2
- net at U8.6: no longer R44.1
- net at Q29.2 (C), R87.2: now also Q30.1 (S), Q30.2 (D)
- net at C18.1, R104.1, RL104.2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: now also Q30.3 (G), Q33.1 (S), Q33.2 (D)
- net at Q27.2 (E), R88.2, U11.2 (-): now also Q33.3 (G)
- net at C21.2, D14.3 (K), R68.2: now also R107.1
- net at Q11.3 (G): now also D19.3 (K)
- new net: Q31.3 (E), Q34.1 (B), Q34.2 (E), R108.1, R89.1
- new net: R103.2, R89.2
- new net: R103.1, R105.1, U15.2 (-)
- new net: Q31.1 (B), U15.6
- new net: R106.1, R107.2
- new net: Q34.3 (C), R106.2
Other:
- note added: "+2.5V"
- note added: "+6.9V from voltage reference probably?"
- note added: "+9V"
- note added: "Blue text are measured voltages on a faulty board"

Commit message: asdf
Parts:
- added D20: BAS21 "JS t", Package_TO_SOT_SMD:SOT-23, symbol Diode:BAS21
- added J7: Conn_02x13_Odd_Even, symbol Connector_Generic:Conn_02x13_Odd_Even
- added R109, R110: 47k, symbol Device:R
- added R111, R113: 2.7k, symbol Device:R
- added R112: 4.7k, symbol Device:R
- added R114, R115: 2.2R, symbol Device:R
- added TP4, TP5: TestPoint, symbol Connector:TestPoint
- Q6: value Q_PMOS_GDS -> 2P50EG
- R31: value 10.2k -> 2.2k
Connections:
- net at Q6.3 (S), RL1.3, RL1.7: now also TP5.1
- net at RL1.4: now also TP4.1
- net at D2.1 (A), M104.6, R26.2: now also RL4.7
- net at Q28.2 (E), R81.1, R82.1: now also R111.2
- net at D9.2 (A), M104.3 (+), R80.1: now also R113.1
- net at C2.1, M104.7 (V+), Q12.1 (B)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: now also D3.1 (A)
- net at C18.1, Q30.3 (G), Q33.1 (S)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: now also R109.2, R110.2, R114.1, R115.1
- net at D17.2 (A), D5.1 (A), D6.1 (K): now also Q12.3 (C), D20.1 (A)
- net at Q28.3 (C): now also M103.13 (V+)
- net at D3.3 (K), R30.2, R31.2: now also J7.20 (Pin_20)
- net at Q104.3 (G1): now also R110.1
- net at M103.4 (-IN): now also R109.1
- new net: R114.2, R115.2
- new net: R111.1, R112.2
- new net: R112.1, R113.2
Other:
- note added: "+16V"
- note added: "-0.8V"
- note added: "-15"
- note added: "0V"
- note added: "29"
- note added: "30V"
- note added: "32V"
- note added: "33V"
- note added: "35V"
- note removed: "+2.5V"
- note removed: "+9V"
- note removed: "11V"
- moved on the sheet: C4, C5, C6, C7, C8, C9, D3, Q10, Q104A, Q104B, Q12, Q5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

Commit message: asdf
Connections:
- net GND: now also Q22.1 (B)
- net at Q16.2 (E), R40.2, R43.1: now also J7.22 (Pin_22)
- net at Q20.1 (B), R47.2: now also D12.3 (K); no longer D12.2 (A)
- no-connect marks 5 -> 3
Other:
- note added: "+3V"
- note added: "-0.3V"
- note added: "-0.47V"
- note added: "-13V"
- note added: "0.6V"
- note added: "4.74V"
- note added: "7.6V"
- note added: "7V"
- note added: "8.24V"
- note added: "8.2V"
- note added: "8.8V"
- note removed: "+16V"
- note removed: "7.5V"
- note removed: "8.19V"
- moved on the sheet: C1, C10, C109, C11, C110, C12, C13, C14, C15, C16, C17, C18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

Commit message: asdf
Parts:
- added D21: BAV99 "A7W", Package_TO_SOT_SMD:SOT-23, symbol Diode:BAV99
- added Q35: BC846 "1DW", symbol Device:Q_NPN_BEC
- added Q36: Q_NJFET_DSG, symbol Device:Q_NJFET_DSG
- added R116: 4.7k, symbol Device:R
- added R117: 6.9k, symbol Device:R_Shunt
- added R118, R119, R120, R121: 2.2k, symbol Device:R
- added TH1: Thermistor_NTC, symbol Device:Thermistor_NTC
- added TP6: TestPoint, symbol Connector:TestPoint
- added U16: LTC1150, Package_SO:SOIC-8_3.9x4.9mm_P1.27mm, symbol Amplifier_Operational:LTC1152
- added U17: LM35-LP, Package_TO_SOT_THT:TO-92_Inline, symbol Sensor_Temperature:LM35-LP
- added unit 2 of U5
Connections:
- net -15V: now also C4.1, Q5.2 (C), Q7.3 (C), R8.1, U4.4 (V-)
- net GND: now also RL3.1, RL3.7
- net at Q6.3 (S), RL1.3, RL1.7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: now also R118.1
- net at R105.2, R44.1, U8.2 (-): now also R117.2
- net at U8.6: now also Q35.1 (B)
- net at U8.7 (V+): now also Q35.3 (C), U17.1 (+V_{S})
- net at Q8.3 (E), R21.2, R23.2: now also NT3.2
- net at NT4.2, Q5.3 (E), R15.2: no longer Q7.2 (E)
- net at Q23.3 (C): now also R116.1
- net at RL2.3: now also C19.1, C20.1
- net at C18.2, C19.2, C20.2: now also R121.2
- net at Q26.1 (B), R75.2: now also R116.2
- net at NT7.2, U7.3 (+): now also U5.6
- net at Q5.1 (B), R15.1: now also Q7.2 (E)
- net at NT5.2: now also TP6.1
- new net: R120.1, R121.1
- new net: Q35.2 (E), R117.1
- new net: R117.3, U16.2 (-)
- new net: Q36.2 (S), R117.4
- new net: R118.2, R119.1
- new net: R119.2, R120.2
- new net: D21.1 (K), Q36.1 (D)
- new net: TH1.1, U17.3 (GND)
- new net: Q36.3 (G), U16.6
Other:
- note added: "Current sinks run even when not in use to keep temperatures constant?"
- note added: "V-Difference between U4 +in and U7 +in sets I-Sink mA?"
- moved on the sheet: C10, C109, C11, C110, C12, C13, C2, C4, C5, C6, C7, C8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

Commit message: asdf
Parts:
- added C25, C26, C27, C28: 10µF Tantal, symbol Device:C_Polarized
- added C29: ?nF Foil, symbol Device:C
- added D22: BAV99 "A7W", Package_TO_SOT_SMD:SOT-23, symbol Diode:BAV99
- added D23: "BUG" or "8U6", symbol Device:D
- added Q37: MMBF4117, symbol Device:Q_NJFET_SDG
- added R122, R125: 1k, symbol Device:R
- added R123, R126: 2.2k, symbol Device:R
- added R124: 100R, symbol Device:R
- added U18: LM337_TO220, Package_TO_SOT_THT:TO-220-3_Vertical, symbol Regulator_Linear:LM337_TO220
- added U19: LTC1150, symbol Amplifier_Operational:LTC1152
Connections:
- net GND: now also C25.1, C26.1, C27.2, C28.1, D23.1 (K), R122.2, R123.2
- net at U5.10: now also U5.7, U19.3 (+)
- net at Q32.1 (B), R94.2: now also R126.1
- net at NT5.2, TP6.1: now also C26.2, C29.1, D22.3 (K), D23.2 (A), R124.2, U18.3 (VO)
- net at U2.2 (VI): now also C28.2, U18.2 (VI)
- net at NT6.2: now also C29.2
- net at NT12.2: now also R125.1
- new net: C25.2, D22.2 (A), R122.1, R123.1, R124.1, U18.1 (ADJ)
- new net: R125.2, U19.2 (-)
- new net: Q37.3 (G), U19.6
Other:
- note added: "-10V"
- note added: "-15V"
- note added: "-19.22V"
- note added: "-8.68V"
- note added: "0.135V"
- note added: "0.82V"
- note added: "11V"
- note added: "4.7V"
- note added: "4.9V"
- note added: "PSUs"
- note added: "higher current sinks"
- note added: "something with Vrefs?"
- note removed: "PSU region probably"
- note removed: "Vref region probably"
- moved on the sheet: C1, C4, C5, C6, C7, C8, C9, D4, Q10, Q23, Q5, Q7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
