File: resistance_board_RE/resistance_board_RE.kicad_sch (KiCad schematic)
At the start: 280 parts, among them J1 Red Wire, J2 Blrown Wire, J3 Yellow Wire, J4 Black Wire, J5 Green Wire, J6 Orange Wire, J7 Conn_02x13_Odd_Even, M103 LTC1052CSW-PBF, M104 MC33071, M203 LTC1052CSW-PBF, Q1 FZT658, Q10 MMBF5485 "6M", Q104 SST404, Q11 MMBF5485 "6M", Q12 BC856 "3DW", Q13 FZT493, Q14 TIP32CG Heatsunk, Q15 FZT658, Q16 BC856 "3DW", Q17 BC846 "1DW", Q18 BC846 "1DW", Q19 BC846 "1DW", Q2 TIP32CG Heatsunk, Q20 BC846 "1DW", Q21 FZT758, Q22 BC846 "1DW", Q23 BC856 "3DW", Q24 BC846 "1DW", Q25 FZT493, Q26 BC846 "1DW", Q27 BC846 "1DW", Q28 BC846 "1DW", Q29 FZT758, Q3 04N80C3, Q30 MMBF4117, Q31 FZT493, Q32 BC856 "3DW", Q33 MMBF4117, Q34 BC846 "1DW", Q35 BC846 "1DW", Q36 Q_NJFET_DSG, Q37 MMBF4117, Q4 FZT758, Q5 TIP32CG Heatsunk, Q6 2P50EG, Q7 BC856 "3DW", Q8 TIP31AG Heatsunk, Q9 BC846 "1DW", U1 PVI5080N, U10 TL071, U11 TL071, U12 TL071, U13 DG408DY+T, U14 DG211, U15 TL071, U16 LTC1150, U17 LM35-LP, U18 LM337_TO220, U19 LTC1150, U2 LM337_TO220, U3 PVI5080N, U4 LTC1150, U5 DG211, U6 TL071, U7 LTC1150, U8 LTC1150, U9 TL071

Commit message: asdf
Parts:
- added C30: 22µF 400V Al, symbol Device:C_Polarized
- added C31: 4.7µF 400V Al, symbol Device:C_Polarized
- added D24: BAS21 "JS t", Package_TO_SOT_SMD:SOT-23, symbol Diode:BAS21
- added D25, D26, D28: BAV99 "A7W", Package_TO_SOT_SMD:SOT-23, symbol Diode:BAV99
- added D27: BZX84-C5V6 "Z3W", Package_TO_SOT_SMD:SOT-23, symbol Diode:BZX84Cxx
- added Q38, Q47: BC846 "1DW", symbol Device:Q_NPN_BEC
- added Q39, Q42: FZT658, symbol Device:Q_NPN_BCE
- added Q40, Q41: FZT758, symbol Device:Q_PNP_BCE
- added Q43, Q44, Q45, Q46: BC856 "3DW", symbol Device:Q_PNP_BEC
- added R127, R128: 330R, symbol Device:R
- added R129, R131, R142, R143, R144: 10k, symbol Device:R
- added R130, R141: 47k, symbol Device:R
- added R132, R133, R137, R138, R139, R140, R146, R147, R148, R149: 100k, symbol Device:R
- added R134, R135, R136: 1M, symbol Device:R
- added R145: 2.2k, symbol Device:R
- added TP7: TestPoint, symbol Connector:TestPoint
- added U20: TL071, symbol Amplifier_Operational:TL071
Connections:
- net +15V: now also Q43.2 (E), R142.1, R143.1, U20.7 (V+)
- net -15V: now also Q41.2 (C), Q42.3 (E), Q46.3 (C), R144.2, U20.4 (V-)
- net GND: now also Q17.2 (E), Q18.2 (E), R48.2, Q38.2 (E), R141.1, R148.1
- net at D20.3 (K): now also D24.1 (A)
- net at R126.2: now also Q38.3 (C)
- net at Q15.2 (C), R97.1, R98.1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: now also D24.3 (K)
- net at RL1.4, TP4.1: now also R128.2
- net at D9.2 (A), M104.3 (+), R113.1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: now also R132.2, U20.3 (+)
- net at C10.2, C11.1, C12.1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: now also R131.2, R132.1, R133.2
- net at Q20.3 (C), R48.1: now also Q38.1 (B)
- net at C24.2, RL4.5: now also D28.3 (K), Q42.2 (C)
- net at C24.1: now also Q42.1 (B), Q45.3 (C), R144.1
- new net: Q39.3 (E), Q47.1 (B), R127.1, TP7.1
- new net: R127.2, R128.1
- new net: R139.1, R140.2
- new net: R138.1, R139.2
- new net: Q43.1 (B), Q44.2 (E), R142.2, R143.2
- new net: R148.2, R149.1
- new net: Q45.1 (B), R129.1, U20.6
- new net: R129.2, R130.1
- new net: C31.1, R140.1
- new net: R135.1, R136.2
- new net: R134.1, R135.2
- new net: Q43.3 (C), Q44.1 (B), R141.2
- new net: D25.1 (K), D26.1 (K), Q44.3 (C)
- new net: D25.3 (K), Q45.2 (E)
- new net: D27.1 (A), Q40.1 (B), R146.2
- new net: Q39.2 (C), Q40.2 (C)
- new net: Q40.3 (E), R145.1
- new net: C30.1, D27.3 (K), R145.2
- new net: Q41.3 (E), Q47.2 (E)
- new net: D28.1 (K), Q39.1 (B), Q47.3 (C), R137.2
- new net: R147.1, R149.2
- new net: R146.1, R147.2
- new net: R137.1, R138.2
- new net: Q46.1 (B), R133.1, R134.2
- new net: D26.3 (K), Q46.2 (E)
- new net: R130.2, R131.1, U20.2 (-)
- new net: Q41.1 (B), R136.1
Other:
- note added: "7.0V"
- note added: "HV Entry likely"
- note removed: "-0.47V"
- moved on the sheet: C24, D17, D20, D8, J4, Q13, Q15, Q20, R32, R33, R71, U13

Commit message: asdf
Parts:
- added TP10, TP11, TP12, TP13, TP8, TP9: TestPoint, symbol Connector:TestPoint
Other:
- note added: "-0.022V"
- note added: "-1.2V"
- note added: "-4.2V"
- note added: "-7.38V"
- note added: "6.9V"

Commit message: asdf
Parts:
- added C32, C33: 1uF Film, symbol Device:C
- added C34: 100nF Film, symbol Device:C
- added C35, C36, C37: 47nF Film, symbol Device:C
- added D29: BZX84-C5V6 "Z3W", Package_TO_SOT_SMD:SOT-23, symbol Diode:BZX84Cxx
- added Q48: BC846 "1DW", symbol Device:Q_NPN_BEC
- added R150: 10k, symbol Device:R
- added R151: 220R, symbol Device:R
- added R152, R153: 10M, symbol Device:R
- C11, C13: value 47nF Foil -> 47nF Film
- C12: value 47nF Foil -> 100nF Film
- R34: value 10M -> 22k
- renumbered U12 to M102
Connections:
- net +15V: now also R35.1
- net -15V: now also R34.2, D29.1 (A)
- net GND: now also R150.2
- net at Q104.1 (S1), Q104.5 (S2): now also Q48.3 (C)
- net at Q104.6 (D2): now also R37.1, C32.1
- net at Q104.7 (G2): now also J3.1 (Pin_1), M103.3 (NC(GUARD)), M103.5 (+IN), M103.6 (NC(GUARD))
- net at L3.1, R3.1, R5.2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: now also R114.2, R115.2, RL101.4
- net at C13.1: now also R79.1, C34.1
- net at C13.2: now also M102.2 (-), C32.2, C34.2, R152.1
- net at M102.3 (+): now also C33.2, R151.1, R153.2
- net at M102.6, R79.2, R80.2: now also R152.2
- net at R34.1: now also Q48.2 (E)
- net at C10.2, C11.1, C12.1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: now also C35.1, C37.1, R153.1; no longer R34.2
- net at R36.1: now also Q104.2 (D1), C33.1
- net at C12.2: now also C11.2, R151.2
- net at R112.1, R113.2: now also C35.2, C36.2
- new net: C36.1, C37.2
- new net: D29.3 (K), Q48.1 (B), R150.1
Other:
- note added: "Displayed: Always?!"
- note added: "Displayed: DCV, ACV, DCI, ACI etc Flipped: Any Ω Range"
- note added: "Displayed: Never?!"
- note added: "Displayed: Normal Flipped: 100 mA excitation"
- note added: "Displayed: Normal Flipped: HiV Ω"
- note added: "Displayed: Normal Flipped: Ω Filt"
- note removed: "30V"
- moved on the sheet: C10, C109, C110, J3, M102, M103, Q104A, Q104B, Q28, R109, R110, R111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

Commit message: asdf
Parts:
- added D30: BAV99 "JYW", Package_TO_SOT_SMD:SOT-23, symbol Diode:BAV99
- added NT14, NT15, NT16, NT17, NT18, NT20, NT21, NT22, NT23, NT24, NT25: NetTie_2, symbol Device:NetTie_2
- added Q49: MMBF4117, symbol Device:Q_NJFET_SDG
- added R154, R155: 1k, symbol Device:R
- added R156, R157, R160: 1.9k, symbol Device:R
- added R158: 20.2k?, symbol Device:R
- added R159: 16.7k?, symbol Device:R
- added U12: DG211, Package_SO:SOIC-16_3.9x9.9mm_P1.27mm, symbol Analog_Switch:DG411xY
- added unit 1 of U5
Connections:
- net at U8.3 (+): now also R155.1
- net at J7.7 (Pin_7): now also R155.2
- net at J7.8 (Pin_8): now also R154.2
- net at U16.3 (+): now also R154.1
- net at RL3.5: now also D30.3 (K)
- new net: NT14.1, NT15.1, R156.2
- new net: NT23.1, NT24.1, R160.1
- new net: NT21.1, NT22.1, R158.1, R159.1, R160.2
- new net: NT25.1, R158.2
- new net: NT16.1, R156.1, R157.1
- new net: NT17.1, NT18.1, R157.2
- new net: NT20.1, R159.2
Other:
- note added: "-4.8V"
- note added: "RN2 Fluke 4345110R measured in circuit"
