File: resistance_board_RE/_autosave-resistance_board_RE.kicad_sch (KiCad schematic)
At the start: 200 parts, among them J1 Red Wire, J2 Blrown Wire, J3 Yellow Wire, J4 Black Wire, J5 Green Wire, J6 Orange Wire, M103 LTC1052CSW-PBF, M104 MC33071, M203 LTC1052CSW-PBF, Q1 FZT658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

Commit message: asdf
Parts:
- added RL4, RL5: TX2-L-12V, symbol Relay:G6KU-2
Connections:
- net at L3.1, R3.1, R5.2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: now also RL4.2
- new net: RL4.3, RL5.2
Other:
- note removed: "Constant current sinks maybe?"
- moved on the sheet: RL102, TP102
